File: boards/twintest/twintest.kicad_sch (KiCad schematic)
At the start: 20 parts, among them J1 USB_C, SW1 SW_Push, U1 STM32F072CBT6, U3 XC6206, U4 USBLC6-2SC6

Commit message: update
Parts:
- removed C10, C11, C13, C16, C7: 100nF, ScottoKeebs_Components:Capacitor_0402, symbol Device:C_Small
- removed C12, C17: 4.7uF, ScottoKeebs_Components:Capacitor_0402, symbol Device:C_Small
- removed C14: 10nF, ScottoKeebs_Components:Capacitor_0402, symbol Device:C_Small
- removed C15, C8, C9: 1uF, ScottoKeebs_Components:Capacitor_0402, symbol Device:C_Small
- removed F1: 500mA, ScottoKeebs_Components:Fuse_0603, symbol Device:Fuse_Small
- removed J1: USB_C, ScottoKeebs_Components:USB_C_HRO_TYPE-C-31-M-12, symbol Connector:USB_C_Receptacle_USB2.0_14P
- removed R1: 10k, ScottoKeebs_Components:Resistor_0402, symbol Device:R_Small
- removed R2, R3: 5.1k, ScottoKeebs_Components:Resistor_0402, symbol Device:R_Small
- removed SW1: SW_Push, ScottoKeebs_Components:Button_TL3342, symbol Switch:SW_Push
- removed U1: STM32F072CBT6, ScottoKeebs_Components:Package_LQFP-48_7x7mm_P0.5, symbol MCU_ST_STM32F0:STM32F072CBTx
- removed U3: XC6206, ScottoKeebs_Components:Voltage_SOT-23, symbol Regulator_Linear:XC6206PxxxMR
- removed U4: USBLC6-2SC6, ScottoKeebs_Components:ESD_SOT-23-6, symbol Power_Protection:USBLC6-2SC6
- added BT2: Battery_Cell, ScottoKeebs_Scotto:Battery, symbol Device:Battery_Cell
- added D1, D10, D11, D12, D13, D14, D15, D16, D17, D18, D19, D2, D20, D21, D22, D23, D24, D25, D26, D27, D3, D4, D5, D6, D7, D8, D9: Diode, ScottoKeebs_Components:Diode_DO-35, symbol ScottoKeebs:Placeholder_Diode
- added H1, H2, H3, H4, H5, H6: Mounting_Hole, ScottoKeebs_Scotto:Standoff_M2x6mm, symbol ScottoKeebs:Placeholder_Mounting_Hole
- added S1, S10, S11, S12, S13, S14, S15, S16, S17, S18, S19, S2, S20, S21, S22, S23, S24, S25, S26, S27, S3, S4, S5, S6, S7, S8, S9: Keyswitch, ScottoKeebs_MX:MX_PCB_1.00u, symbol ScottoKeebs:Placeholder_Keyswitch
- added SW1: Switch, ScottoKeebs_Components:Switch_MSK12C02, symbol ScottoKeebs:Placeholder_Switch
- added U1, U2: Nice_Nano_V2, ScottoKeebs_MCU:Nice_Nano_V2, symbol ScottoKeebs:MCU_Nice_Nano_V2
Connections:
- new net: D24.2 (A), S24.2
- new net: D12.2 (A), S12.2
- new net: D27.2 (A), S27.2
- new net: D17.2 (A), S17.2
- new net: D18.2 (A), S18.2
- new net: D9.2 (A), S9.2
- new net: D21.2 (A), S21.2
- new net: D5.2 (A), S5.2
- new net: D15.2 (A), S15.2
- new net: D26.2 (A), S26.2
- new net: BT2.1 (+), SW1.2
- new net: D7.2 (A), S7.2
- new net: D3.2 (A), S3.2
- new net: D16.2 (A), S16.2
- new net: D10.2 (A), S10.2
- new net: D14.2 (A), S14.2
- new net: D8.2 (A), S8.2
- new net: D19.2 (A), S19.2
- new net: D20.2 (A), S20.2
- new net: D13.2 (A), S13.2
- new net: D25.2 (A), S25.2
- new net: D23.2 (A), S23.2
- new net: D22.2 (A), S22.2
- new net: D2.2 (A), S2.2
- new net: D4.2 (A), S4.2
- new net: D11.2 (A), S11.2
- new net: D6.2 (A), S6.2
- new net: D1.2 (A), S1.2
- new net battery +: SW1.1, U1.24 (B+), U2.24 (B+)
- new net battery -: BT2.2 (-), U1.1, U2.1
- new net collumn 1: S1.1, S13.1, S19.1, S7.1, U1.5 (2), U2.5 (2)
- new net collumn 2: S14.1, S2.1, S20.1, S8.1, U1.6 (3), U2.6 (3)
- new net collumn 3: S15.1, S21.1, S3.1, S9.1, U1.7 (4), U2.7 (4)
- new net collumn 4: S10.1, S16.1, S22.1, S25.1, S4.1, U1.8 (5), U2.8 (5)
- new net collumn 5: S11.1, S17.1, S23.1, S26.1, S5.1, U1.9 (6), U2.9 (6)
- new net collumn 6: S12.1, S18.1, S24.1, S27.1, S6.1, U1.10 (7), U2.10 (7)
- new net row 1: D1.1 (K), D2.1 (K), D3.1 (K), D4.1 (K), D5.1 (K), D6.1 (K), U1.20 (21), U2.20 (21)
- new net row 2: D10.1 (K), D11.1 (K), D12.1 (K), D7.1 (K), D8.1 (K), D9.1 (K), U1.19 (20), U2.19 (20)
- new net row 3: D13.1 (K), D14.1 (K), D15.1 (K), D16.1 (K), D17.1 (K), D18.1 (K), U1.18 (19), U2.18 (19)
- new net row 4: D19.1 (K), D20.1 (K), D21.1 (K), D22.1 (K), D23.1 (K), D24.1 (K), U1.17 (18), U2.17 (18)
- new net row 5: D25.1 (K), D26.1 (K), D27.1 (K), U1.16 (15), U2.16 (15)
Other:
- note removed: "Bootloader Button"
- note removed: "Connector"
- note removed: "Controller"
- note removed: "Decoupling Capacitors"
- note removed: "ESD Protection"
- note removed: "Matrix"
- note removed: "Mounting Holes"
- note removed: "Other"
- note removed: "Power Flags"
- note removed: "STM32F072CBT6"
- note removed: "USB-C"
- note removed: "Voltage Step Down"
